File: pp_bob_input.sch (KiCad schematic (older format))
At the start: 16 parts, among them P1 2X8, P2 2X5, P3 2X4, P4 13X2, U1 74LVC245, U2 74LVC245, U3 74LS541

Commit message: Redraw layout
Parts:
- removed P1: 2X8, Pin_Headers:Pin_Header_Straight_2x08_Pitch2.54mm, symbol CONN_02X08
- removed P2: 2X5, Pin_Headers:Pin_Header_Straight_2x05_Pitch2.54mm, symbol CONN_02X05
- removed P3: 2X4, Pin_Headers:Pin_Header_Straight_2x04_Pitch2.54mm, symbol CONN_02X04
- added J_IN_1, J_IN_2, J_IN_3, J_IN_4: ST_1x04, Connectors_Terminal_Blocks:TerminalBlock_Pheonix_PT-3.5mm_4pol, symbol Screw_Terminal_1x04
- added J_IN_5, J_OUT_2: ST_1x12, Connectors_Terminal_Blocks:TerminalBlock_Pheonix_PT-3.5mm_12pol, symbol Screw_Terminal_1x12
- added J_IN_6: ST_1x03, Connectors_Terminal_Blocks:TerminalBlock_Pheonix_PT-3.5mm_3pol, symbol Screw_Terminal_1x03
- U3: symbol 74LS541 -> 74LS541-RESCUE-pp_bob_input
Connections:
- wire segments 146 -> 189
- no-connect marks 6 -> 5

Commit message: Initial V0.3 commit
Parts:
- removed J_IN_5: ST_1x12, Connectors_Terminal_Blocks:TerminalBlock_Pheonix_PT-3.5mm_12pol, symbol Screw_Terminal_1x12
- removed J_IN_6: ST_1x03, Connectors_Terminal_Blocks:TerminalBlock_Pheonix_PT-3.5mm_3pol, symbol Screw_Terminal_1x03
- removed PCE_1: 1X4, Pin_Headers:Pin_Header_Straight_1x04_Pitch2.54mm, symbol CONN_01X04
- added J_IN_5: ST_1x15, w_conn_pt-1,5:pt_1,5-15-3,5-h, symbol Screw_Terminal_1x15
- added RN1: 4k7, Resistors_THT:R_Array_SIP9, symbol R_Network08
- added RN4: 4k7, Resistors_THT:R_Array_SIP5, symbol R_Network04
- added SEL_1, SEL_2, SEL_3, SEL_4: 1X3, Pin_Headers:Pin_Header_Straight_1x03_Pitch2.54mm, symbol CONN_01X03
- J_IN_1, J_IN_2, J_IN_3, J_IN_4: footprint Connectors_Terminal_Blocks:TerminalBlock_Pheonix_PT-3.5mm_4pol -> w_conn_pt-1,5:pt_1,5-4-3,5-h
- J_OUT_2: footprint Connectors_Terminal_Blocks:TerminalBlock_Pheonix_PT-3.5mm_12pol -> w_conn_pt-1,5:pt_1,5-12-3,5-h
- R1: footprint Resistors_SMD:R_1210_HandSoldering -> Resistors_THT:R_Axial_DIN0204_L3.6mm_D1.6mm_P7.62mm_Horizontal
- RN2: value 10k -> 3k3
- RN3: renamed from RN1; value 10k -> 4k7; footprint Resistors_THT:R_Array_SIP4 -> Resistors_THT:R_Array_SIP9; symbol R_Network03 -> R_Network08
- renumbered PPWRIN_1 to PWRIN_1, PPWRSEL_1 to PWRSEL_1
Connections:
- net IN-03 is gone; now on net IN-02: J_IN_1.3, U1.17 (B2)
- net SCHP is gone; now on net CHIP_ENABLE: P4.26 (P22)
- net +3V3: now also SEL_2.3 (P3)
- net +5V: now also J_IN_5.1, J_IN_5.10, J_IN_5.13, J_IN_5.4, J_IN_5.7, SEL_1.3 (P3), SEL_3.3 (P3), SEL_4.3 (P3)
- net GND: now also U3.2 (A0), U3.3 (A1), U3.4 (A2), U3.5 (A3), J_IN_5.12, J_IN_5.15, J_IN_5.3, J_IN_5.6, J_IN_5.9, SEL_1.1 (P1), SEL_2.1 (P1), SEL_3.1 (P1), SEL_4.1 (P1); no longer RN2.1 (common)
- net IN-02: now also RN1.8 (R7), RN1.9 (R8)
- net IN-04: now also RN1.7 (R6)
- net IN-05: now also RN1.6 (R5)
- net IN-06: now also RN1.5 (R4)
- net IN-07: now also RN1.4 (R3)
- net IN-08: now also RN1.3 (R2)
- net IN-09: now also RN1.2 (R1)
- net IN-10: now also RN3.9 (R8), J_IN_5.2
- net IN-11: now also RN3.8 (R7), J_IN_5.5
- net IN-12: now also RN3.7 (R6), J_IN_5.8
- net IN-13: now also RN3.6 (R5), J_IN_5.11
- net IN-15: now also RN3.5 (R4), J_IN_5.14
- net OUT-01: now also RN4.5 (R4)
- net OUT-14: now also RN4.4 (R3)
- net OUT-16: now also RN4.3 (R2)
- net OUT-17: now also RN4.2 (R1)
- net at RN3.1 (common): now also SEL_3.2 (P2)
- new net: RN2.1 (common), SEL_2.2 (P2)
- new net: RN1.1 (common), SEL_1.2 (P2)
- new net: RN4.1 (common), SEL_4.2 (P2)
Other:
- note removed: "External +5V power"
- note removed: "chip enable select"
- moved on the sheet: J_IN_1, J_IN_2, J_IN_3, J_IN_4, RN2

Commit message: Layout modded to max output board
Parts:
- removed J_IN_5: ST_1x15, w_conn_pt-1,5:pt_1,5-15-3,5-h, symbol Screw_Terminal_1x15
- added J_IN_5, J_IN_6, J_IN_7, J_IN_8, J_IN_9, J_OUT_6, J_OUT_7, J_OUT_8: ST_1x03, w_conn_pt-1,5:pt_1,5-3-3,5-h, symbol Screw_Terminal_1x03
- J_OUT_5: renamed from J_OUT_2; value ST_1x12 -> ST_1x03; footprint w_conn_pt-1,5:pt_1,5-12-3,5-h -> w_conn_pt-1,5:pt_1,5-3-3,5-h; symbol Screw_Terminal_1x12 -> Screw_Terminal_1x03
Connections:
- net +5V: now also J_IN_5.1, J_IN_6.1, J_IN_7.1, J_IN_8.1, J_IN_9.1, J_OUT_6.1, J_OUT_7.1, J_OUT_8.1; no longer J_OUT_5.10, J_OUT_5.4, J_OUT_5.7
- net GND: now also J_IN_5.3, J_IN_6.3, J_IN_7.3, J_IN_8.3, J_IN_9.3, J_OUT_6.3, J_OUT_7.3, J_OUT_8.3; no longer J_OUT_5.12, J_OUT_5.6, J_OUT_5.9
- net IN-10: now also J_IN_5.2
- net IN-11: now also J_IN_6.2
- net IN-12: now also J_IN_7.2
- net IN-13: now also J_IN_8.2
- net IN-15: now also J_IN_9.2
- net OUT-14: now also J_OUT_6.2; no longer J_OUT_5.5
- net OUT-16: now also J_OUT_7.2; no longer J_OUT_5.8
- net OUT-17: now also J_OUT_8.2; no longer J_OUT_5.11
Changed lines of the file:
@@
 $EndComp
 $Comp
-L Screw_Terminal_1x12 J_OUT_2
+L Screw_Terminal_1x03 J_OUT_5
 U 1 1 58F01EB1
-P 6350 2400
-F 0 "J_OUT_2" H 6350 3675 50  0000 C TNN
-F 1 "ST_1x12" V 6200 2400 50  0000 C TNN
-F 2 "w_conn_pt-1,5:pt_1,5-12-3,5-h" H 6350 1975 50  0001 C CNN
-F 3 "" H 6325 2600 50  0001 C CNN
-	1    6350 2400
+P 6350 1500
+F 0 "J_OUT_5" H 6125 1725 50  0000 C TNN
+F 1 "ST_1x03" V 6200 1375 50  0000 C TNN
+F 2 "w_conn_pt-1,5:pt_1,5-3-3,5-h" H 6350 1075 50  0001 C CNN
+F 3 "" H 6325 1700 50  0001 C CNN
+	1    6350 1500
 	1    0    0    -1
 $EndComp
@@
 NoConn ~ 8200 2275
 NoConn ~ 8200 2175
-$Comp
-L Screw_Terminal_1x15 J_IN_5
-U 1 1 58F030F1
-P 1175 2000
-F 0 "J_IN_5" H 1175 3250 50  0000 C TNN
-F 1 "ST_1x15" V 1025 2000 50  0000 C TNN
-F 2 "w_conn_pt-1,5:pt_1,5-15-3,5-h" H 1175 775 50  0001 C CNN
-F 3 "" H 1150 3000 50  0001 C CNN
-	1    1175 2000
-	1    0    0    -1
-$EndComp
 $Comp
 L R_Network08 RN1
@@
 	2150 4175 3100 4175
 Connection ~ 9700 2475
-Text Label 2750 5150 0    50   ~ 0
+$Comp
+L Screw_Terminal_1x03 J_IN_5
+U 1 1 58FDD36D
+P 1175 1100
+F 0 "J_IN_5" H 1000 1325 50  0000 C TNN
+F 1 "ST_1x03" V 1025 975 50  0000 C TNN
+F 2 "w_conn_pt-1,5:pt_1,5-3-3,5-h" H 1175 675 50  0001 C CNN
+F 3 "" H 1150 1300 50  0001 C CNN
+	1    1175 1100
+	1    0    0    -1
+$EndComp
+$Comp
+L Screw_Terminal_1x03 J_IN_6
+U 1 1 58FDD8CB
+P 1175 1700
+F 0 "J_IN_6" H 1000 1925 50  0000 C TNN
+F 1 "ST_1x03" V 1025 1575 50  0000 C TNN
+F 2 "w_conn_pt-1,5:pt_1,5-3-3,5-h" H 1175 1275 50  0001 C CNN
+F 3 "" H 1150 1900 50  0001 C CNN
+	1    1175 1700
+	1    0    0    -1
+$EndComp
+$Comp
+L Screw_Terminal_1x03 J_IN_7
+U 1 1 58FDDFC7
+P 1175 2300
+F 0 "J_IN_7" H 1000 2525 50  0000 C TNN
+F 1 "ST_1x03" V 1025 2175 50  0000 C TNN
+F 2 "w_conn_pt-1,5:pt_1,5-3-3,5-h" H 1175 1875 50  0001 C CNN
+F 3 "" H 1150 2500 50  0001 C CNN
+	1    1175 2300
+	1    0    0    -1
+$EndComp
+$Comp
+L Screw_Terminal_1x03 J_IN_8
+U 1 1 58FDE5AC
+P 1175 2900
+F 0 "J_IN_8" H 1000 3125 50  0000 C TNN
+F 1 "ST_1x03" V 1025 2775 50  0000 C TNN
+F 2 "w_conn_pt-1,5:pt_1,5-3-3,5-h" H 1175 2475 50  0001 C CNN
+F 3 "" H 1150 3100 50  0001 C CNN
+	1    1175 2900
+	1    0    0    -1
+$EndComp
+$Comp
+L Screw_Terminal_1x03 J_IN_9
+U 1 1 58FDE6B1
+P 1175 3500
+F 0 "J_IN_9" H 1000 3725 50  0000 C TNN
+F 1 "ST_1x03" V 1025 3375 50  0000 C TNN
+F 2 "w_conn_pt-1,5:pt_1,5-3-3,5-h" H 1175 3075 50  0001 C CNN
+F 3 "" H 1150 3700 50  0001 C CNN
+	1    1175 3500
+	1    0    0    -1
+$EndComp
+$Comp
+L Screw_Terminal_1x03 J_OUT_6
+U 1 1 58FE2DE0
+P 6350 2100
+F 0 "J_OUT_6" H 6125 2325 50  0000 C TNN
+F 1 "ST_1x03" V 6200 1975 50  0000 C TNN
+F 2 "w_conn_pt-1,5:pt_1,5-3-3,5-h" H 6350 1675 50  0001 C CNN
+F 3 "" H 6325 2300 50  0001 C CNN
+	1    6350 2100
+	1    0    0    -1
+$EndComp
+$Comp
+L Screw_Terminal_1x03 J_OUT_7
+U 1 1 58FE2F74
+P 6350 2700
+F 0 "J_OUT_7" H 6125 2925 50  0000 C TNN
+F 1 "ST_1x03" V 6200 2575 50  0000 C TNN
+F 2 "w_conn_pt-1,5:pt_1,5-3-3,5-h" H 6350 2275 50  0001 C CNN
+F 3 "" H 6325 2900 50  0001 C CNN
+	1    6350 2700
+	1    0    0    -1
+$EndComp
+$Comp
+L Screw_Terminal_1x03 J_OUT_8
+U 1 1 58FE367E
+P 6350 3300
+F 0 "J_OUT_8" H 6125 3525 50  0000 C TNN
+F 1 "ST_1x03" V 6200 3175 50  0000 C TNN
+F 2 "w_conn_pt-1,5:pt_1,5-3-3,5-h" H 6350 2875 50  0001 C CNN
+F 3 "" H 6325 3500 50  0001 C CNN
+	1    6350 3300
+	1    0    0    -1
+$EndComp
+Text Label 2750 5150 0    40   ~ 0
 IN-03
 $EndSCHEMATC
